File: v1/hardware/kicad/gps/gps.kicad_pcb (KiCad board)
At the start: 2 copper layers, 1 part, among them U1 ublox_SAM-M8Q

Commit message: update
Parts:
- added BT1: Battery_Cell, Battery:BatteryHolder_Keystone_1058_1x2032, B.Cu at (333.8, -67.6)
- added BT2: Battery_Cell, Battery:BatteryHolder_Keystone_1042_1x18650, F.Cu at (317.0, -35.3)
- added J1: Conn_01x14_Female, Connector_PinSocket_2.54mm:PinSocket_1x14_P2.54mm_Vertical, F.Cu at (355.6, -31.0)
- added J3: Conn_01x04_Female, Connector_PinSocket_2.54mm:PinSocket_1x04_P2.54mm_Vertical, F.Cu at (339.2, -81.7)
- added J4: Conn_01x06_Female, Connector_PinSocket_2.54mm:PinSocket_1x06_P2.54mm_Vertical, F.Cu at (348.2, -51.3)
- added J5: Conn_Coaxial, Connector_Coaxial:SMA_Molex_73251-1153_EdgeMount_Horizontal, F.Cu at (348.7, -86.6)
- added SW1: SW_Push, Button_Switch_THT:SW_Tactile_SPST_Angled_PTS645Vx58-2LFS, F.Cu at (360.7, -78.5)
- added SW2: SW_Push, Button_Switch_THT:SW_Tactile_SPST_Angled_PTS645Vx58-2LFS, F.Cu at (360.7, -68.1)
- added SW3: SW_Push, Button_Switch_THT:SW_Tactile_SPST_Angled_PTS645Vx58-2LFS, F.Cu at (360.7, -57.9)
- added SW4: SW_Push, Button_Switch_THT:SW_Tactile_SPST_Angled_PTS645Vx58-2LFS, F.Cu at (360.7, -47.8)
- added U2: RFM95HW, RF_Module:HOPERF_RFM9XW_SMD, F.Cu at (345.2, -69.8)
- moved U1 288.5 mm to (316.0, -91.7)
Connections:
- net Net-(U1-Pad1) renamed GND
- U1 pad 17: (no net) -> 3V3
- U1 pad 2: (no net) -> 3V3
- U1 pad 3: (no net) -> Net-(BT1-Pad1)
Other:
- board outline added: 58.4 x 120.5 mm
